Commit message: Improve support for d435 and add missing mesh files

File: turtlebot_description/urdf/sensors/d435.urdf.xacro (robot description, xacro)
@@ -4,6 +4,6 @@
   <xacro:include filename="$(find turtlebot_description)/urdf/turtlebot_properties.urdf.xacro"/>
   <!-- Mount and camera parameters -->
-  <xacro:property name="pole_px" value="-0.103" />
-  <xacro:property name="pole_py" value="-0.098"/>
+  <xacro:property name="pole_px" value="-0.055" />
+  <xacro:property name="pole_py" value="-0.12"/>
   <xacro:property name="pole_pz" value="0.269" />
   <xacro:property name="d435_bracket_end_offset_py" value="0.02" />
@@ -14,7 +14,7 @@
   <xacro:property name="d435_bracket_length"    value="0.176" />
   <xacro:property name="d435_bracket_width"     value="0.0285" />
-  <xacro:property name="d435_cam_offset_px" value="-0.017" />
-  <xacro:property name="d435_cam_offset_py" value="0.024" />
-  <xacro:property name="d435_cam_offset_pz" value="0.005" />
+  <xacro:property name="d435_cam_offset_px" value="0.0" />
+  <xacro:property name="d435_cam_offset_py" value="0.1" />
+  <xacro:property name="d435_cam_offset_pz" value="0.015" />
   <xacro:property name="d435_cam_rgb_px" value="0.005"/>
   <xacro:property name="d435_cam_rgb_py" value="0.018"/>

Commit message: Change the camera placement

File: turtlebot_description/urdf/sensors/d435.urdf.xacro (robot description, xacro)
@@ -3,15 +3,4 @@
   <xacro:include filename="$(find turtlebot_description)/urdf/turtlebot_gazebo.urdf.xacro"/>
   <xacro:include filename="$(find turtlebot_description)/urdf/turtlebot_properties.urdf.xacro"/>
-  <!-- Mount and camera parameters -->
-  <xacro:property name="pole_px" value="-0.055" />
-  <xacro:property name="pole_py" value="-0.12"/>
-  <xacro:property name="pole_pz" value="0.269" />
-  <xacro:property name="d435_bracket_end_offset_py" value="0.02" />
-  <xacro:property name="d435_bracket_end_offset_pz" value="0" />
-  <xacro:property name="d435_bracket_end_width"     value="0.026" />
-  <xacro:property name="d435_bracket_offset_py" value="0.010" />
-  <xacro:property name="d435_bracket_offset_pz" value="0.010" />
-  <xacro:property name="d435_bracket_length"    value="0.176" />
-  <xacro:property name="d435_bracket_width"     value="0.0285" />
   <xacro:property name="d435_cam_offset_px" value="0.0" />
   <xacro:property name="d435_cam_offset_py" value="0.1" />
@@ -22,56 +11,8 @@
   <xacro:property name="d435_cam_depth_offset" value="0.01"/>
   <xacro:macro name="sensor_d435" params="parent">
-    <!--
-    ==  Mount and camera body joints & links ==
-    -->
-    <!-- right bracket end -->
-    <joint name="bracket_end_right_joint" type="fixed">
-      <origin xyz="${pole_px} ${pole_py} ${pole_pz}" rpy="0 0 0"/>
-      <parent link="${parent}"/>
-      <child link="bracket_end_right" />
-    </joint>
-    <link name="bracket_end_right">
-    <visual>
-       <origin xyz="${-d435_bracket_end_width/2} ${d435_bracket_end_offset_py} ${d435_bracket_end_offset_pz}" rpy="0 0 ${-M_PI/2}"/>
-        <geometry>
-         <mesh filename="package://turtlebot_description/meshes/sensors/d435_bracket_end.stl" scale="0.001 0.001 0.001"/>
-        </geometry>
-        <xacro:insert_block name="material_dark_grey" />
-      </visual>
-    </link>
-    <!-- center main bracket -->
-    <joint name="bracket_joint" type="fixed">
-      <origin xyz="${d435_bracket_width/2} ${d435_bracket_offset_py} ${d435_bracket_offset_pz}" rpy="0 0 0"/>
-      <parent link="bracket_end_right"/>
-      <child link="bracket" />
-    </joint>
-    <link name="bracket">
-    <visual>
-       <origin xyz="0 0 0" rpy="0 0 ${M_PI/2}"/>
-        <geometry>
-         <mesh filename="package://turtlebot_description/meshes/sensors/d435_bracket.stl" scale="0.001 0.001 0.001"/>
-        </geometry>
-        <xacro:insert_block name="material_dark_grey" />
-      </visual>
-    </link>
-    <!-- left bracket end -->
-    <joint name="bracket_end_left_joint" type="fixed">
-      <origin xyz="${-d435_bracket_width/2} ${d435_bracket_length - d435_bracket_offset_py} ${-d435_bracket_offset_pz}" rpy="0 0 0"/>
-      <parent link="bracket"/>
-      <child link="bracket_end_left" />
-    </joint>
-    <link name="bracket_end_left">
-    <visual>
-       <origin xyz="${d435_bracket_end_width/2} 0 ${-d435_bracket_end_offset_pz}" rpy="0 0 ${M_PI/2}"/>
-        <geometry>
-         <mesh filename="package://turtlebot_description/meshes/sensors/d435_bracket_end.stl" scale="0.001 0.001 0.001"/>
-        </geometry>
-        <xacro:insert_block name="material_dark_grey" />
-      </visual>
-    </link>
     <!-- camera body -->
     <joint name="camera_joint" type="fixed">
-      <origin xyz="${d435_cam_offset_px} ${d435_cam_offset_py} ${d435_cam_offset_pz}" rpy="0 0 0"/>
-      <parent link="bracket"/>
+      <origin xyz="-0.105 0 0.197" rpy="0 0 ${M_PI}"/>
+      <parent link="${parent}"/>
       <child link="camera_link" />
     </joint>
@@ -128,5 +69,5 @@
     </joint>
     <link name="camera_depth_optical_frame"/>
-  	<!-- Simulation sensor -->
+	<!-- Simulation sensor -->
     <xacro:turtlebot_sim_3dsensor/>
   </xacro:macro>

Commit message: Update 'egokituz' stack design & camera placement

File: turtlebot_description/urdf/sensors/d435.urdf.xacro (robot description, xacro)
@@ -13,5 +13,5 @@
     <!-- camera body -->
     <joint name="camera_joint" type="fixed">
-      <origin xyz="-0.105 0 0.197" rpy="0 0 ${M_PI}"/>
+      <origin xyz="0.155 0 0.16" rpy="0 0 0"/>
       <parent link="${parent}"/>
       <child link="camera_link" />

File: turtlebot_description/urdf/stacks/egokituz.urdf.xacro (robot description, xacro)
@@ -3,5 +3,5 @@
   Hexagon stacks
  -->
-<robot name="stack_egokituz" xmlns:xacro="http://ros.org/wiki/xacro">
+<robot name="stack_hexagons" xmlns:xacro="http://ros.org/wiki/xacro">
   <xacro:include filename="$(find turtlebot_description)/urdf/common_properties.urdf.xacro"/>
   <!-- Xacro properties -->
@@ -65,60 +65,4 @@
     </link>
   </xacro:macro>
-  <xacro:macro name="stack_top_pole" params="parent number x_loc y_loc z_loc roll=0.0 pitch=0.0 yaw=0.0">
-    <joint name="pole_top_${number}_joint" type="fixed">
-      <origin xyz="${x_loc} ${y_loc} ${z_loc}" rpy="${roll} ${pitch} ${yaw}"/>
-      <parent link="${parent}"/>
-      <child link="pole_top_${number}_link"/>
-    </joint>
-    <link name="pole_top_${number}_link">
-      <visual>
-        <origin xyz=" 0 0 0" rpy="0 0 0"/>
-        <geometry>
-          <mesh filename="package://turtlebot_description/meshes/stacks/hexagons/pole_top.dae"/>
-        </geometry>
-      </visual>
-      <collision>
-        <origin xyz="0 0 0" rpy="0 0 0"/>
-        <geometry>
-          <cylinder length="0.2032" radius="0.006"/>
-        </geometry>
-      </collision>
-      <inertial>
-        <mass value="0.060"/>
-        <origin xyz="0 0 0"/>
-        <inertia ixx="0.000206991" ixy="0.0" ixz="0.0"
-                 iyy="0.000206991" iyz="0.0"
-                 izz="0.000001080"/>
-      </inertial>
-    </link>
-  </xacro:macro>
-  <xacro:macro name="stack_3d_sensor_pole" params="parent number x_loc y_loc z_loc roll=0.0 pitch=0.0 yaw=0.0">
-    <joint name="pole_kinect_${number}_joint" type="fixed">
-      <origin xyz="${x_loc} ${y_loc} ${z_loc}" rpy="${roll} ${pitch} ${yaw}"/>
-      <parent link="${parent}"/>
-      <child link="pole_kinect_${number}_link"/>
-    </joint>
-    <link name="pole_kinect_${number}_link">
-      <visual>
-        <origin xyz="0 0 0" rpy="0 0 0"/>
-        <geometry>
-          <mesh filename="package://turtlebot_description/meshes/stacks/hexagons/pole_kinect.dae" />
-        </geometry>
-      </visual>
-      <collision>
-        <origin xyz="0 0 0" rpy="0 0 0"/>
-        <geometry>
-          <cylinder length="0.0936" radius="0.006"/>
-        </geometry>
-      </collision>
-      <inertial>
-        <mass value="0.020"/>
-        <origin xyz="0 0 0"/>
-        <inertia ixx="0.000014782" ixy="0.0" ixz="0.0"
-                 iyy="0.000014782" iyz="0.0"
-                 izz="0.000000360"/>
-      </inertial>
-    </link>
-  </xacro:macro>
   <!--
     Stack macro - all the components relative transforms are made with respect
@@ -128,11 +72,11 @@
   <xacro:macro name="stack_hexagons" params="parent">
     <xacro:stack_bottom_pole parent="${parent}" number="0" x_loc= "0.120" y_loc= "0.082" z_loc="0.1028"/>
-    <!-- <xacro:stack_bottom_pole parent="${parent}" number="1" x_loc= "0.055" y_loc= "0.120" z_loc="0.1028"/> -->
+    <xacro:stack_bottom_pole parent="${parent}" number="1" x_loc= "0.055" y_loc= "0.120" z_loc="0.1028"/>
     <xacro:stack_bottom_pole parent="${parent}" number="2" x_loc="-0.055" y_loc= "0.120" z_loc="0.1028"/>
     <xacro:stack_bottom_pole parent="${parent}" number="3" x_loc= "0.120" y_loc="-0.082" z_loc="0.1028"/>
-    <!-- <xacro:stack_bottom_pole parent="${parent}" number="4" x_loc= "0.055" y_loc="-0.120" z_loc="0.1028"/> -->
+    <xacro:stack_bottom_pole parent="${parent}" number="4" x_loc= "0.055" y_loc="-0.120" z_loc="0.1028"/>
     <xacro:stack_bottom_pole parent="${parent}" number="5" x_loc="-0.055" y_loc="-0.120" z_loc="0.1028"/>
     <joint name="plate_bottom_joint" type="fixed">
-      <origin xyz="0.02364 0.0 0.1814" rpy="0 0 0"/>
+      <origin xyz="0.02364 0.0 0.1306" rpy="0 0 0"/>
       <parent link="${parent}"/>
       <child link="plate_bottom_link"/>
@@ -159,9 +103,8 @@
       </inertial>
     </link>
-    <xacro:stack_middle_pole parent="${parent}" number="0" x_loc= "0.12" y_loc= "0.082" z_loc="0.1580"/>
-    <xacro:stack_middle_pole parent="${parent}" number="1" x_loc= "-0.055" y_loc="0.12" z_loc="0.1580"/>
-    <xacro:stack_middle_pole parent="${parent}" number="2" x_loc="0.12" y_loc= "-0.082" z_loc="0.1580"/>
-    <xacro:stack_middle_pole parent="${parent}" number="3" x_loc="-0.055" y_loc="-0.12" z_loc="0.1580"/>
-    <!--
+    <xacro:stack_middle_pole parent="${parent}" number="0" x_loc= "0.0381" y_loc= "0.1505" z_loc="0.1640"/>
+    <xacro:stack_middle_pole parent="${parent}" number="1" x_loc= "0.0381" y_loc="-0.1505" z_loc="0.1640"/>
+    <xacro:stack_middle_pole parent="${parent}" number="2" x_loc="-0.0381" y_loc= "0.1505" z_loc="0.1640"/>
+    <xacro:stack_middle_pole parent="${parent}" number="3" x_loc="-0.0381" y_loc="-0.1505" z_loc="0.1640"/>
     <joint name="plate_middle_joint" type="fixed">
       <origin xyz="-0.01364 0.0 0.1874" rpy="0 0 0"/>
@@ -173,5 +116,5 @@
         <origin xyz="0 0 0" rpy="0 0 0"/>
         <geometry>
-          <mesh filename="package://turtlebot_description/meshes/stacks/hexagons/plate_middle.dae"/>
+          <mesh filename="package://turtlebot_description/meshes/stacks/hexagons/plate_top.dae"/>
         </geometry>
       </visual>
@@ -179,5 +122,5 @@
         <origin xyz="0.01364 0.0 0.0" rpy="0 0 0"/>
         <geometry>
-          <mesh filename="package://turtlebot_description/meshes/stacks/hexagons/plate_simple.stl"
+          <mesh filename="package://turtlebot_description/meshes/stacks/hexagons/plate_top.stl"
                 scale="${M_SCALE} ${M_SCALE} ${M_SCALE}"/>
         </geometry>
@@ -191,38 +134,4 @@
       </inertial>
     </link>
-    <xacro:stack_top_pole parent="${parent}" number="0" x_loc= "0.0381" y_loc= "0.1505" z_loc="0.2920"/>
-    <xacro:stack_top_pole parent="${parent}" number="1" x_loc= "0.0381" y_loc="-0.1505" z_loc="0.2920"/>
-    <xacro:stack_top_pole parent="${parent}" number="2" x_loc="-0.0381" y_loc= "0.1505" z_loc="0.2920"/>
-    <xacro:stack_top_pole parent="${parent}" number="3" x_loc="-0.0381" y_loc="-0.1505" z_loc="0.2920"/>
-    <xacro:stack_3d_sensor_pole parent="${parent}" number="0" x_loc="-0.1024" y_loc= "0.098" z_loc="0.2372"/>
-    <xacro:stack_3d_sensor_pole parent="${parent}" number="1" x_loc="-0.1024" y_loc="-0.098" z_loc="0.2372"/>
-    <joint name="plate_top_joint" type="fixed">
-      <origin xyz="-0.01364 0.0  0.3966" rpy="0 0 0"/>
-      <parent link="${parent}"/>
-      <child link="plate_top_link"/>
-    </joint>
-    <link name="plate_top_link">
-      <visual>
-        <origin xyz="0 0 0" rpy="0 0 0"/>
-        <geometry>
-          <mesh filename="package://turtlebot_description/meshes/stacks/hexagons/plate_top.dae"/>
-        </geometry>
-      </visual>
-      <collision>
-        <origin xyz="0.01364 0 0" rpy="0 0 0"/>
-        <geometry>
-          <mesh filename="package://turtlebot_description/meshes/stacks/hexagons/plate_simple.stl"
-                scale="${M_SCALE} ${M_SCALE} ${M_SCALE}"/>
-        </geometry>
-      </collision>
-      <inertial>
-        <mass value="0.520"/>
-        <origin xyz="0 0 0"/>
-        <inertia ixx="0.003328" ixy="0.0" ixz="0.0"
-                 iyy="0.003328" iyz="0.0"
-                 izz="0.006656" />
-      </inertial>
-    </link>
-    -->
   </xacro:macro>
 </robot>
