Commit message: Change ydlidar placement and improve support

File: turtlebot_description/robots/kobuki_egokituz_d435_x4.urdf.xacro (robot description, xacro)
@@ -14,4 +14,4 @@
   <xacro:stack_hexagons parent="base_link"/>
   <xacro:sensor_d435    parent="base_link"/>
-  <xacro:ydlidar_x4 name="ydlidar" base="base_link" pose_xyz="0.252 0 0.066" pose_rpy="0 0 ${-M_PI/2-6/180*M_PI}" />
+  <xacro:ydlidar_x4 name="ydlidar" base="base_link" pose_xyz="-0.0095 0.0095 0.225" pose_rpy="0 0 ${-6/180*M_PI}" />
 </robot>

File: turtlebot_description/urdf/stacks/egokituz.urdf.xacro (robot description, xacro)
@@ -122,5 +122,5 @@
         <origin xyz="0.01364 0.0 0.0" rpy="0 0 0"/>
         <geometry>
-          <mesh filename="package://turtlebot_description/meshes/stacks/hexagons/plate_top.stl"
+          <mesh filename="package://turtlebot_description/meshes/stacks/hexagons/plate_top.dae"
                 scale="${M_SCALE} ${M_SCALE} ${M_SCALE}"/>
         </geometry>
